File: hardware/programmer_reva.sch (EAGLE design)
At the start: 2 parts

Commit message: final hardware files, already sent to fab
Parts:
- added U$2: LOGO, circuitpython-logo:LOGO
Changed lines of the file:
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@@
 <part name="GND2" library="SparkFun-Aesthetics" deviceset="GND" device=""/>
 <part name="GND3" library="SparkFun-Aesthetics" deviceset="GND" device=""/>
+<part name="U$2" library="circuitpython-logo" deviceset="LOGO" device=""/>
 </parts>
 <sheets>
@@
 <instance part="GND2" gate="1" x="33.02" y="165.1"/>
 <instance part="GND3" gate="1" x="53.34" y="165.1"/>
+<instance part="U$2" gate="G$1" x="101.6" y="203.2"/>
 </instances>
 <busses>
