File: hardware/M0_Express_ekho_shield.sch (EAGLE design)
At the start: 56 parts, among them SW1 KMR2, U2 AP2112-3.3, U7 LTC2058, U9 ADP1613, X3 microUSB, X4 32.768

Commit message: final schematic
Parts:
- removed C12, C3: 0.1uF, tiny_passives:C-EU0603
- removed R10: 1.91M, tiny_passives:R-EU0603
- removed R11: 22k, tiny_passives:R-EU0603
- removed R12: 10k, tiny_passives:R-EU0603
- removed U$3: SCREW_CONNECTOR-2PIN', BaseApp:SCREW_CONNECTOR-2PIN'
- removed U7: LTC2058, sorber:LTC2058
- added OP1: LT1797, LT1797:LT1797
- added R3: 470, SparkFun-Passives:RESISTOR0805-RES
- added R6: 3M, tiny_passives:R-EU0603
- added R7: 1M, tiny_passives:R-EU0603
- R8: value 470 -> 2.2k; device SparkFun-Passives:RESISTOR0805-RES -> tiny_passives:R-EU0603; DIGIKEY (none) -> 311-40.2KLRCT-ND
- R9: value 4.22M -> 1k; DIGIKEY P2.0MJCT-ND -> 311-40.2KLRCT-ND
Connections:
- removed net AMPOUT: R11.1, R8.1, U7.OUTA
- removed net INA-: R11.2, R12.2, U7.-INA
- removed net VS_AMP: JP1.2, U7.-INB, U7.OUTB
- new net HARVESTER_IN: OP1.OUT, R3.1, R8.2
- new net N$5: OP1.IN-, R8.1, R9.2
- net AVCC_SET: now also OP1.V+; no longer C3.1, U7.V+
- net GND: now also OP1.V-, R7.2, R9.1; no longer C12.2, C3.2, R10.2, R12.1, U$3.1, U7.V-
- net LOAD_V+: now also JP1.2, R3.2, R6.1; no longer R8.2, R9.1, U$3.2
- net VDAC: now also OP1.IN+; no longer C12.1, U7.+INA
- net VS_ADC: now also R6.2, R7.1; no longer R10.1, R9.2, U7.+INB
Other:
- note added: "1/4 Division"
- note added: "Gain=3.2"
- note removed: "1/3.2 Division"
- note removed: "Emulation Control (DAC)"
- note removed: "GAIN = 3.2"
- note removed: "Voltage Sense"

Commit message: final ekho hardware done
Parts:
- removed SW1: KMR2, microbuilder:SWITCH_TACT_SMT4.6X2.8
- removed X3: microUSB, microbuilder:USB_MICRO_20329_V2
- added C2: 1uF, microbuilder:CAP_CERAMIC0603_NO
- added J1: MF-CON-MICROUSB-RIGHT, MF_Connectors:USB_MICRO_RIGHT
- added S3: TL1015AF, eswitch:TL1015AF
- JP12, JP13: device SparkFun-Connectors:M02 -> SparkFun-Connectors:M02LOCK
- U$14: DIGIKEY (none) -> ATSAMD51J19A-MU-ND; MPN (none) -> ATSAMD51J19A-MU
Connections:
- removed net N$1: R5.1, U$14G$2.PB05/I5/AIN7
- removed net N$2: R2.1, U$14G$2.PB04/I4/AIN6
- new net LED1: R2.1, U$14G$1.PA12/I12/I2C/SERCOM2.0+4.1
- new net LED2: R5.1, U$14G$1.PA13/I13/I2C/SERCOM2.1+4.0
- net !RESET: now also S3.2; no longer SW1.P, SW1.P1
- net AVCC_SET: now also C2.1
- net D+: now also J1.D+; no longer X3.D+
- net D-: now also J1.D-; no longer X3.D-
- net GND: now also C2.2, J1.GND, J1.SLD, S3.1, S3.GND, S3.GND@, S3.GND@@, S3.GND@@@; no longer SW1.S, SW1.S1, X3.GND
- net TDI/RX_DEBUG: now also U$14G$1.PA05/I5/AIN5/VOUT1/SERCOM0.1; no longer U$14G$2.PB03/I3/AIN15/SERCOM5.1
- net TDO/TX_DEBUG: now also U$14G$1.PA04/I4/VREFB/AIN4/SERCOM0.0; no longer U$14G$2.PB02/I2/AIN14/SERCOM5.0
- net VBUS: now also J1.5V; no longer X3.VBUS
- net VS_ADC: now also U$14G$1.PA11/I11/AIN11/SERCOM0+2.3/I2SDO; no longer U$14G$1.PA04/I4/VREFB/AIN4/SERCOM0.0

Commit message: can measure current and communicate/takeover the M0 kind of like a debugger
Parts:
- added C3: 0.1uF, tiny_passives:C-EU0603
- added C4: 1.0uF, tiny_passives:C-EU0603
- added R10: 10, SparkFun-Passives:RESISTOR0805-RES
- added U1: INA225, ina225:INA225
- R3: value 470 -> 100
Connections:
- removed net A0: JP_AD.1
- removed net A1: JP_AD.2
- removed net A2: JP_AD.3
- removed net A3: JP_AD.4
- removed net LOAD_V+: JP1.2, R3.2, R6.1
- new net CSG0: U$14G$1.PA21/I5/SERCOM3+5.3/I2SDO, U1.GS0
- new net CSG1: U$14G$1.PA20/I4/SERCOM3+5.2/I2SFS0, U1.GS1
- new net CS_ADC: U$14G$1.PA15/I15/SERCOM2+4.3, U1.OUT
- new net HIGH_LOAD_V+: R10.1, R3.2, U1.IN+
- new net LOW_LOAD_V+: JP1.2, R10.2, R6.1, U1.IN-
- net +3V3: now also C3.1, C4.1, U1.VS
- net GND: now also C3.2, C4.2, U1.GND, U1.REF
- net LED1: now also U$14G$2.PB10/I10/SERCOM4.2/I2SDI; no longer U$14G$1.PA12/I12/I2C/SERCOM2.0+4.1
- net LED2: now also U$14G$2.PB11/I11/SERCOM4.3/I2SFS1; no longer U$14G$1.PA13/I13/I2C/SERCOM2.1+4.0
- net NV_CLK: now also U$14G$1.PA16/I2C/I0/SERCOM1.0+3.1
- net NV_CS: now also U$14G$1.PA18/I2/SERCOM1+3.2
- net NV_READ: now also U$14G$2.PB16/I0/SERCOM5.0/I2SCK0
- net NV_SIMO: now also U$14G$1.PA17/I2C/I1/SERCOM1.1+3.0
- net NV_SOMI: now also U$14G$1.PA19/I3/SERCOM1+3.3
- net NV_WRITE: now also U$14G$2.PB17/SERCOM5.1/I2SMCK0
- net VS_ADC: now also U$14G$1.PA14/I14/SERCOM2+4.2; no longer U$14G$1.PA11/I11/AIN11/SERCOM0+2.3/I2SDO
Other:
- note added: "A0"
- note added: "A1"
- note added: "A2"
- note added: "A3"
- note added: "Current Sense"
- note added: "Emulator Output"
- note added: "Harvester Connection"
- note added: "Sense Resistor"
- note added: "Voltage Sense"
- moved on the sheet: C1, C15, C16, C18, C19, C2, C6, C8, D+, D-, D1, D4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
